Commit message: feat(osmag): implement robust passage resolution, corridor A* scaling, and topometric world synchronization

File: lidarbot_ws/src/lidarbot/lidarbot_gz/urdf/sensors.xacro (robot description, xacro)
@@ -146,5 +146,5 @@
     <parent link="base_link"/>
     <child link="lidar_link"/>
-    <origin xyz="0.1385 0.0095 0.08" rpy="0 0 ${-pi/2}"/>
+    <origin xyz="0.1385 0.0095 0.08" rpy="0 0 0"/>
     <axis xyz="0 0 1"/>
   </joint>
